File: another-space-pcb/another-space-pcb.kicad_pcb (KiCad board)
At the start: 2 copper layers, 271.5 x 76.2 mm, 105 parts, among them SW1 RotaryEncoder_Switch, SW2 RotaryEncoder_Switch, U1 ProMicro

Commit message: Updated pcb silkscreen
Other:
- board text added: "another space 1.0.1 (2024)"
- board text removed: "another space 1.0 (2024) github.com/mhzkb"
